File: helix.sch (KiCad schematic (older format))
At the start: 136 parts, among them J1 MJ-4PP-9, P3 OLED, Q1 2SC2712, Q2 2SC2712, SW1 SW_PUSH, SW10 SW_PUSH, SW11 SW_PUSH, SW12 SW_PUSH, SW13 SW_PUSH, SW14 SW_PUSH, SW15 SW_PUSH, SW16 SW_PUSH, SW17 SW_PUSH, SW18 SW_PUSH, SW19 SW_PUSH, SW2 SW_PUSH, SW20 SW_PUSH, SW21 SW_PUSH, SW22 SW_PUSH, SW23 SW_PUSH, SW24 SW_PUSH, SW25 SW_PUSH, SW26 SW_PUSH, SW27 SW_PUSH, SW28 SW_PUSH, SW29 SW_PUSH, SW3 SW_PUSH, SW30 SW_PUSH, SW31 SW_PUSH, SW32 SW_PUSH, SW33 Reset, SW34 SW_PUSH, SW35 SW_PUSH, SW36 SW_PUSH, SW37 SW_PUSH, SW38 SW_PUSH, SW39 SW_PUSH, SW4 SW_PUSH, SW40 SW_PUSH, SW41 SW_PUSH, SW42 SW_PUSH, SW43 SW_PUSH, SW44 SW_PUSH, SW45 SW_PUSH, SW46 SW_PUSH, SW47 SW_PUSH, SW48 SW_PUSH, SW49 SW_PUSH, SW5 SW_PUSH, SW50 SW_PUSH, SW51 SW_PUSH, SW52 SW_PUSH, SW53 SW_PUSH, SW54 SW_PUSH, SW55 SW_PUSH, SW56 SW_PUSH, SW57 SW_PUSH, SW58 SW_PUSH, SW59 SW_PUSH, SW6 SW_PUSH, SW60 SW_PUSH, SW61 SW_PUSH, SW62 SW_PUSH, SW63 SW_PUSH, SW64 SW_PUSH, SW65 SW_PUSH, SW7 SW_PUSH, SW8 SW_PUSH, SW9 SW_PUSH, U1 ProMicro, U34 74HC4051, U35 74HC4051, U36 AD8616, U37 AD8616, U38 ProMicro

Commit message: ノイズ対策＆nizとvarmiloを同じリポジトリにした
Parts:
- removed JP27, JP28: MountingHole_Pad, phi-kbd-library-master:THSmallest, symbol Mechanical:MountingHole_Pad
- added JP35, JP36, JP37, JP38, JP39, JP40, JP41, JP42: MountingHole_Pad, phi-kbd-library-master:THSmallest, symbol Mechanical:MountingHole_Pad
- added L1, L10, L11, L12, L13, L14, L15, L16, L17, L18, L19, L2, L20, L21, L22, L23, L24, L25, L26, L27, L28, L29, L3, L30, L31, L32, L4, L5, L6, L7, L8, L9: SK6812MINI, ec_helix:SK6812MINI_narrow-irreversible2, symbol kbd:SK6812MINI
- R16, R22: value 51kΩ -> 51-100kΩ
- SW1, SW10, SW11, SW12, SW13, SW14, SW15, SW16, SW17, SW18, SW19, SW2, SW20, SW21, SW22, SW23, SW24, SW25, SW26, SW27, SW28, SW29, SW3, SW30, SW31, SW32, SW34, SW35, SW36, SW37, SW38, SW39, SW4, SW40, SW41, SW42, SW43, SW44, SW45, SW46, SW47, SW48, SW49, SW5, SW50, SW51, SW52, SW53, SW54, SW55, SW56, SW57, SW58, SW59, SW6, SW60, SW61, SW62, SW63, SW64, SW65, SW7, SW8, SW9: footprint ec_helix:niz -> ec_helix:MX_Hotswap-1.00u-irreversible
- U1, U38: footprint ec_helix:ProMicro -> kbd:ProMicro_v3.5
- renumbered R7 to R11, R9 to R12, R28 to R26, R26 to R27, R27 to R28, R30 to R29, R29 to R30, R11 to R6, R6 to R7, R12 to R9
Connections:
- net a_ is gone; now on net a: C1.1, R14.1, R15.1, U34.3 (A)
- net GND: now also L1.2 (VSS), L10.2 (VSS), L11.2 (VSS), L12.2 (VSS), L13.2 (VSS), L14.2 (VSS), L15.2 (VSS), L16.2 (VSS), L17.2 (VSS), L18.2 (VSS), L19.2 (VSS), L2.2 (VSS), L20.2 (VSS), L21.2 (VSS), L22.2 (VSS), L23.2 (VSS), L24.2 (VSS), L25.2 (VSS), L26.2 (VSS), L27.2 (VSS), L28.2 (VSS), L29.2 (VSS), L3.2 (VSS), L30.2 (VSS), L31.2 (VSS), L32.2 (VSS), L4.2 (VSS), L5.2 (VSS), L6.2 (VSS), L7.2 (VSS), L8.2 (VSS), L9.2 (VSS)
- net LED: now also L6.3 (DIN); no longer JP25.1, U1.1 (TX)
- net SCL: no longer JP23.1, U1.6 (SCL)
- net SDA: no longer JP20.1, U1.5 (SDA)
- net VCC: now also L1.4 (VDD), L10.4 (VDD), L11.4 (VDD), L12.4 (VDD), L13.4 (VDD), L14.4 (VDD), L15.4 (VDD), L16.4 (VDD), L17.4 (VDD), L18.4 (VDD), L19.4 (VDD), L2.4 (VDD), L20.4 (VDD), L21.4 (VDD), L22.4 (VDD), L23.4 (VDD), L24.4 (VDD), L25.4 (VDD), L26.4 (VDD), L27.4 (VDD), L28.4 (VDD), L29.4 (VDD), L3.4 (VDD), L30.4 (VDD), L31.4 (VDD), L32.4 (VDD), L4.4 (VDD), L5.4 (VDD), L6.4 (VDD), L7.4 (VDD), L8.4 (VDD), L9.4 (VDD)
- net a0: now also R30.1, R6.1, U34.5 (A5), U35.1 (A4); no longer R29.1, R7.1, U34.13 (A0), U35.5 (A5)
- net a1: now also R27.1, R7.1, U34.13 (A0), U35.14 (A1); no longer R11.1, R28.1, U34.14 (A1), U35.15 (A2)
- net a2: now also R26.1, U35.12 (A3); no longer R27.1, U35.14 (A1)
- net a3: now also R9.1, U34.2 (A6); no longer R12.1, U34.12 (A3)
- net a4: now also R29.1, U35.5 (A5); no longer R30.1, U35.1 (A4)
- net a5: now also R11.1, U34.14 (A1); no longer R6.1, U34.5 (A5)
- net a6: now also R12.1, R28.1, U34.12 (A3), U35.15 (A2); no longer R26.1, R9.1, U34.2 (A6), U35.12 (A3)
- net adc: now also R13.2, R16.2, U36.1, U38.13 (B6), JP42.1; no longer U1.13 (B6)
- net adc_: now also U1.13 (B6), JP40.1; no longer R13.2, R16.2, U36.1, U38.13 (B6)
- net charge: now also R17.1, U38.14 (B2), JP41.1; no longer U1.14 (B2)
- net charge_: now also U1.14 (B2), JP39.1; no longer R17.1, U38.14 (B2)
- net col00: no longer JP1.1, U1.7 (D4)
- net col01: no longer JP2.1, U1.8 (C6)
- net col02: no longer JP3.1, U1.9 (D7)
- net col03: no longer JP12.1, U1.10 (E6)
- net col04: no longer JP13.1, U1.11 (B4)
- net data: no longer JP22.1, JP26.1
- net row0: now also U34.11 (S0), U38.20 (F4), JP36.1; no longer U1.20 (F4)
- net row0_: now also JP22.1, U1.20 (F4); no longer U34.11 (S0), U38.20 (F4)
- net row1: now also U34.10 (S1), U38.19 (F5), JP37.1; no longer U1.19 (F5)
- net row1_: now also JP26.1, U1.19 (F5); no longer U34.10 (S1), U38.19 (F5)
- net row2: now also U34.9 (S2), U38.18 (F6), JP38.1; no longer U1.18 (F6)
- net row2_: now also U1.18 (F6), JP35.1; no longer U34.9 (S2), U38.18 (F6)
- net at R16.1, R18.1, U36.2 (-): now also R22.1, R24.1, U37.2 (-)
- net at R14.2, U36.3 (+): now also R20.2, U37.3 (+)
- net at Q2.3 (C), R21.2: now also Q1.3 (C), R15.2
- net at Q2.1 (B), R23.2: now also Q1.1 (B), R17.2
- new net: L5.3 (DIN), L6.1 (DOUT)
- new net: L4.3 (DIN), L5.1 (DOUT)
- new net: L3.3 (DIN), L4.1 (DOUT)
- new net: L2.3 (DIN), L3.1 (DOUT)
- new net: L1.3 (DIN), L2.1 (DOUT)
- new net: L1.1 (DOUT), L7.3 (DIN)
- new net: L7.1 (DOUT), L8.3 (DIN)
- new net: L8.1 (DOUT), L9.3 (DIN)
- new net: L10.3 (DIN), L9.1 (DOUT)
- new net: L10.1 (DOUT), L11.3 (DIN)
- new net: L11.1 (DOUT), L12.3 (DIN)
- new net: L12.1 (DOUT), L18.3 (DIN)
- new net: L17.3 (DIN), L18.1 (DOUT)
- new net: L16.3 (DIN), L17.1 (DOUT)
- new net: L15.3 (DIN), L16.1 (DOUT)
- new net: L14.3 (DIN), L15.1 (DOUT)
- new net: L13.3 (DIN), L14.1 (DOUT)
- new net: L13.1 (DOUT), L19.3 (DIN)
- new net: L19.1 (DOUT), L20.3 (DIN)
- new net: L20.1 (DOUT), L21.3 (DIN)
- new net: L21.1 (DOUT), L22.3 (DIN)
- new net: L22.1 (DOUT), L23.3 (DIN)
- new net: L23.1 (DOUT), L24.3 (DIN)
- new net: L24.1 (DOUT), L25.3 (DIN)
- new net: L26.3 (DIN), L27.1 (DOUT)
- new net: L27.3 (DIN), L28.1 (DOUT)
- new net: L28.3 (DIN), L29.1 (DOUT)
- new net: L29.3 (DIN), L30.1 (DOUT)
- new net: L30.3 (DIN), L31.1 (DOUT)
- new net: L31.3 (DIN), L32.1 (DOUT)
- new net: L25.1 (DOUT), L32.3 (DIN)
- new net LED_: JP25.1, U1.1 (TX)
- new net SCL_: JP23.1, U1.6 (SCL)
- new net SDA_: JP20.1, U1.5 (SDA)
- new net col00_: JP1.1, U1.7 (D4)
- new net col01_: JP2.1, U1.8 (C6)
- new net col02_: JP3.1, U1.9 (D7)
- new net col03_: JP12.1, U1.10 (E6)
- new net col04_: JP13.1, U1.11 (B4)
- no-connect marks 9 -> 10
Other:
- moved on the sheet: C2, JP26, Q2, R19, R20, R21, R22, R23, R24, U37A, U37B
